File: analyze-logic.kicad_pcb (KiCad board)
At the start: 0 parts

Commit message: added board and begin with traces
Parts:
- added C1: 10u, Capacitor_SMD:C_0603_1608Metric, F.Cu at (37.8, 89.2)
- added C10: 100n, Capacitor_SMD:C_0402_1005Metric, F.Cu at (37.3, 81.5)
- added C11: 100n, Capacitor_SMD:C_0402_1005Metric, F.Cu at (37.3, 29.2)
- added C12: 100n, Capacitor_SMD:C_0402_1005Metric, F.Cu at (29.8, 13.3)
- added C13: 100n, Capacitor_SMD:C_0402_1005Metric, F.Cu at (37.2, 13.3)
- added C14: 100n, Capacitor_SMD:C_0402_1005Metric, F.Cu at (29.5, 55.8)
- added C15: 100n, Capacitor_SMD:C_0402_1005Metric, F.Cu at (29.5, 73.0)
- added C16: 100n, Capacitor_SMD:C_0402_1005Metric, F.Cu at (37.1, 55.8)
- added C17: 100n, Capacitor_SMD:C_0402_1005Metric, F.Cu at (37.2, 20.8)
- added C18: 100n, Capacitor_SMD:C_0402_1005Metric, F.Cu at (29.5, 64.2)
- added C2: 10u, Capacitor_SMD:C_0603_1608Metric, F.Cu at (35.8, 96.2)
- added C3: 100n, Capacitor_SMD:C_0402_1005Metric, F.Cu at (29.6, 29.3)
- added C4: 100n, Capacitor_SMD:C_0402_1005Metric, F.Cu at (37.2, 37.5)
- added C5: 100n, Capacitor_SMD:C_0402_1005Metric, F.Cu at (37.1, 64.2)
- added C6: 100n, Capacitor_SMD:C_0402_1005Metric, F.Cu at (29.7, 20.7)
- added C7: 100n, Capacitor_SMD:C_0402_1005Metric, F.Cu at (29.5, 81.6)
- added C8: 100n, Capacitor_SMD:C_0402_1005Metric, F.Cu at (37.2, 73.2)
- added C9: 100n, Capacitor_SMD:C_0402_1005Metric, F.Cu at (29.7, 37.4)
- added D1: LED, Diode_SMD:D_0603_1608Metric, F.Cu at (30.8, 96.2)
- added J1: Input 0 - 7, Connector_IDC:IDC-Header_2x08_P2.54mm_Vertical, F.Cu at (54.8, 36.9)
- added J2: Input 8 - 15, Connector_IDC:IDC-Header_2x08_P2.54mm_Vertical, F.Cu at (54.5, 79.9)
- added J3: Connector Oscilloscope, Connector_IDC:IDC-Header_2x25_P2.54mm_Vertical, F.Cu at (7.25, 81.4)
- added R1: 100R, Resistor_SMD:R_0402_1005Metric, F.Cu at (34.4, 40.1)
- added R10: 100R, Resistor_SMD:R_0402_1005Metric, F.Cu at (26.8, 16.1)
- added R11: 100R, Resistor_SMD:R_0402_1005Metric, F.Cu at (34.3, 75.8)
- added R12: 100R, Resistor_SMD:R_0402_1005Metric, F.Cu at (26.7, 58.5)
- added R13: 100R, Resistor_SMD:R_0402_1005Metric, F.Cu at (26.7, 32.0)
- added R14: 100R, Resistor_SMD:R_0402_1005Metric, F.Cu at (34.2, 16.1)
- added R15: 100R, Resistor_SMD:R_0402_1005Metric, F.Cu at (26.7, 75.8)
- added R16: 100R, Resistor_SMD:R_0402_1005Metric, F.Cu at (34.3, 58.5)
- added R17: 100R, Resistor_SMD:R_0402_1005Metric, F.Cu at (12.2, 80.0)
- added R18: 5k, Resistor_SMD:R_0402_1005Metric, F.Cu at (33.0, 95.8)
- added R2: 100R, Resistor_SMD:R_0402_1005Metric, F.Cu at (26.8, 23.7)
- added R3: 100R, Resistor_SMD:R_0402_1005Metric, F.Cu at (34.2, 84.2)
- added R4: 100R, Resistor_SMD:R_0402_1005Metric, F.Cu at (26.7, 67.0)
- added R5: 100R, Resistor_SMD:R_0402_1005Metric, F.Cu at (26.7, 40.3)
- added R6: 100R, Resistor_SMD:R_0402_1005Metric, F.Cu at (34.4, 23.6)
- added R7: 100R, Resistor_SMD:R_0402_1005Metric, F.Cu at (26.7, 84.2)
- added R8: 100R, Resistor_SMD:R_0402_1005Metric, F.Cu at (34.3, 67.0)
- added R9: 100R, Resistor_SMD:R_0402_1005Metric, F.Cu at (34.3, 32.0)
- added REF**: MountingHole_3.2mm_M3_no_Mask, ownLib:MountingHole_3.2mm_M3_no_Mask, F.Cu at (6.00, 6.00)
- added REF**: MountingHole_3.2mm_M3_no_Mask, ownLib:MountingHole_3.2mm_M3_no_Mask, F.Cu at (54.0, 6.00)
- added REF**: MountingHole_3.2mm_M3_no_Mask, ownLib:MountingHole_3.2mm_M3_no_Mask, F.Cu at (6.00, 94.0)
- added REF**: MountingHole_3.2mm_M3_no_Mask, ownLib:MountingHole_3.2mm_M3_no_Mask, F.Cu at (54.0, 94.0)
- added RN1: 100R, Resistor_SMD:R_Array_Convex_8x0602, F.Cu at (45.1, 27.8)
- added RN2: 100R, Resistor_SMD:R_Array_Convex_8x0602, F.Cu at (45.0, 71.0)
- added U1: MC33375ST-3.3T3G, Package_TO_SOT_SMD:SOT-223, F.Cu at (41.8, 93.8)
- added U10: SN65LVDS1DBV, Package_TO_SOT_SMD:SOT-23-5, F.Cu at (36.8, 32.0)
- added U11: SN65LVDS1DBV, Package_TO_SOT_SMD:SOT-23-5, F.Cu at (29.2, 16.1)
- added U12: SN65LVDS1DBV, Package_TO_SOT_SMD:SOT-23-5, F.Cu at (36.7, 75.8)
- added U13: SN65LVDS1DBV, Package_TO_SOT_SMD:SOT-23-5, F.Cu at (29.1, 58.5)
- added U14: SN65LVDS1DBV, Package_TO_SOT_SMD:SOT-23-5, F.Cu at (29.1, 32.0)
- added U15: SN65LVDS1DBV, Package_TO_SOT_SMD:SOT-23-5, F.Cu at (36.8, 16.1)
- added U16: SN65LVDS1DBV, Package_TO_SOT_SMD:SOT-23-5, F.Cu at (29.1, 75.8)
- added U17: SN65LVDS1DBV, Package_TO_SOT_SMD:SOT-23-5, F.Cu at (36.7, 58.5)
- added U2: SN65LVDS1DBV, Package_TO_SOT_SMD:SOT-23-5, F.Cu at (36.8, 40.2)
- added U3: SN65LVDS1DBV, Package_TO_SOT_SMD:SOT-23-5, F.Cu at (29.2, 23.3)
- added U4: SN65LVDS1DBV, Package_TO_SOT_SMD:SOT-23-5, F.Cu at (36.8, 84.2)
- added U5: SN65LVDS1DBV, Package_TO_SOT_SMD:SOT-23-5, F.Cu at (29.1, 67.0)
- added U6: SN65LVDS1DBV, Package_TO_SOT_SMD:SOT-23-5, F.Cu at (29.1, 40.2)
- added U7: SN65LVDS1DBV, Package_TO_SOT_SMD:SOT-23-5, F.Cu at (36.8, 23.6)
- added U8: SN65LVDS1DBV, Package_TO_SOT_SMD:SOT-23-5, F.Cu at (29.1, 84.3)
- added U9: SN65LVDS1DBV, Package_TO_SOT_SMD:SOT-23-5, F.Cu at (36.7, 67.0)
Routing:
- net VCC: track 0.00 -> 28.3 mm
- net /Di9: track 0.00 -> 23.9 mm
- net /Di1: track 0.00 -> 23.6 mm
- net /Di14: track 0.00 -> 19.7 mm
- net /Di6: track 0.00 -> 19.2 mm
- net /Di11: track 0.00 -> 17.8 mm
- net /Di3: track 0.00 -> 17.5 mm
- net /Di0: track 0.00 -> 17.1 mm
- net /Di8: track 0.00 -> 16.9 mm
- net /Di4: track 0.00 -> 15.3 mm
- net /Di12: track 0.00 -> 15.2 mm
- net /Di15: track 0.00 -> 13.5 mm
- net /Di7: track 0.00 -> 12.1 mm
- net Net-(J1-Pad2): track 0.00 -> 11.9 mm
- net Net-(J1-Pad16): track 0.00 -> 11.6 mm
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Other:
- board outline added: 60 x 100 mm
- copper layers 0 -> 4

Commit message: finished board, updated gitignore
Parts:
- added G***: LOGO, ownLib:LogoMate7x7, F.Cu at (13.6, 11.7)
- moved D1 4.65 mm to (33.5, 92.5), turned to 180 degrees
- moved R17 3.22 mm to (11.6, 83.2), turned to 90 degrees
- moved C1 3.11 mm to (36.3, 92.0), turned to -90 degrees
- moved R18 1.05 mm to (32.9, 94.7), turned to 90 degrees
- moved R2 0.39 mm to (26.9, 23.3)
- moved R7 0.06 mm to (26.7, 84.3)
Routing:
- net VCC: track 28.3 -> 206.7 mm, vias 0 -> 17
- net /D15+: track 0.00 -> 56.5 mm
- net /D15-: track 0.00 -> 53.5 mm
- net +4V: track 4.53 -> 56.4 mm
- net /D10-: track 0.00 -> 49.6 mm, vias 0 -> 1
- net /D13+: track 0.00 -> 48.8 mm
- net /D8-: track 0.00 -> 47.3 mm
- net /D10+: track 0.00 -> 46.8 mm
- net /D14+: track 0.00 -> 46.2 mm
- net /D13-: track 0.00 -> 45.9 mm
- net /D8+: track 0.00 -> 44.9 mm, vias 0 -> 1
- net /D0-: track 0.00 -> 44.7 mm, vias 0 -> 1
- net /D14-: track 0.00 -> 43.4 mm
- net /D7+: track 0.00 -> 42.7 mm
- net /D0+: track 0.00 -> 42.0 mm, vias 0 -> 2
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- added copper zone on B.Cu, net GND
- added copper zone on F.Cu, net GND
- added copper zone on In1.Cu, net GND
- added copper zone on In2.Cu, net GND
Other:
- board text added: "Ch 0...7 GND"
- board text added: "Ch 8...15 GND"
- board text added: "LogicProbe v0.1"
- board text added: "Oscilloscope"
- board text added: "https://github.com/useless-branch - 2022"
- board text added: "pwr ok"
